Commit message: .

File: robot/ros2_ws/src/robot_description/urdf/robot.urdf.xacro (robot description, xacro)
@@ -55,8 +55,7 @@
     <xacro:body_visual mesh_file="spacer_5.stl"/>
     <xacro:body_visual mesh_file="spacer_7.stl"/>
-    <!-- Camera va ga camera chi la visual. camera_link van do
+    <!-- Camera + ga la mot visual assembly. camera_link van do
          orbbec_bringup publish de tranh hai nguon TF trung nhau. -->
-    <xacro:assembly_visual mesh_file="camera_mount.stl" material="dark_grey"/>
-    <xacro:assembly_visual mesh_file="camera_body.stl" material="black"/>
+    <xacro:assembly_visual mesh_file="camera_assembly.stl" material="black"/>
     <!-- Collision = box don gian (khong dung mesh) de Gazebo/ODE dung va cham
          NHANH. Mesh chi tiet lam physics cham vai phut trong VM. -->

File: robot/ros2_ws/src/robot_description/urdf/robot_expanded_hw.urdf (robot description, URDF)
Before this commit: robot amr_robot, 14 links, 13 joints
Links:
- link base_link: geometry collision box size=0.802199951 0.562799988 0.421100037; visual mesh filename=package://robot_description/meshes/body_end_shell_1.stl scale=0.001 0.001 0.001
Joints:
- joint sonar1_link_joint: origin xyz=0.4013235275 0.284999692 0.0 rpy=0 0 0.78539816340 -> xyz=0.4010999755 0.28144996699999997 0.0 rpy=0 0 0.7853981634
- joint sonar2_link_joint: origin xyz=0.4013235275 -0.281226626 0.0 rpy=0 0 -0.78539816340 -> xyz=0.4010999755 -0.281350021 0.0 rpy=0 0 -0.7853981634
- joint sonar3_link_joint: origin xyz=-0.4040990795 0.284999692 0.0 rpy=0 0 2.35619449019 -> xyz=-0.4010999755 0.28144996699999997 0.0 rpy=0 0 2.35619449019
- joint sonar4_link_joint: origin xyz=-0.4040990795 -0.281226626 0.0 rpy=0 0 -2.35619449019 -> xyz=-0.4010999755 -0.281350021 0.0 rpy=0 0 -2.35619449019

File: robot/ros2_ws/src/robot_description/urdf/robot_expanded_sim.urdf (robot description, URDF)
Before this commit: robot amr_robot, 14 links, 13 joints
Links:
- link base_link: geometry collision box size=0.802199951 0.562799988 0.421100037; visual mesh filename=package://robot_description/meshes/body_end_shell_1.stl scale=0.001 0.001 0.001
Joints:
- joint sonar1_link_joint: origin xyz=0.4013235275 0.284999692 0.0 rpy=0 0 0.78539816340 -> xyz=0.4010999755 0.28144996699999997 0.0 rpy=0 0 0.7853981634
- joint sonar2_link_joint: origin xyz=0.4013235275 -0.281226626 0.0 rpy=0 0 -0.78539816340 -> xyz=0.4010999755 -0.281350021 0.0 rpy=0 0 -0.7853981634
- joint sonar3_link_joint: origin xyz=-0.4040990795 0.284999692 0.0 rpy=0 0 2.35619449019 -> xyz=-0.4010999755 0.28144996699999997 0.0 rpy=0 0 2.35619449019
- joint sonar4_link_joint: origin xyz=-0.4040990795 -0.281226626 0.0 rpy=0 0 -2.35619449019 -> xyz=-0.4010999755 -0.281350021 0.0 rpy=0 0 -2.35619449019
