Commit message: robot: calibrate the real robot's LiDAR yaw (base_link -> lidar_link)
The URDF mounted lidar_link at yaw 0, but on the real robot the scan is
rotated by about -12.75 deg relative to base_link:

- LiDAR + wheel distance only (no AMCL, no map): in the straight E-W
  corridor the wall angle in the scan differs from the true heading to the
  walls (from lateral drift per metre driven) by -12.6, -13.3, -12.6 and
  -12.5 deg over 4 passes (2026-10-13 and 2026-10-15, both directions, old
  and new STM32 firmware). Scan handedness checked: in-place turns rotate
  the scene by the wheel yaw change (-25.5 vs -26.6, +151.5 vs +150.7 deg).
- Offline AMCL replays (isolated ROS domain, same params, map and data):
  median lateral error -0.09..-0.20 m at yaw 0 (matching the online runs),
  -0.03..+0.04 m (p90 <= 0.06 m) at -12.75 deg, and -0.33..-0.95 m at
  +12.75 deg. Scan points within 10 cm of a map wall: corridor 29-41 % ->
  65-77 %, corner 9-29 % -> 33-55 %.

This bias made the robot drive 0.27-0.39 m left of the corridor centre on
every run, down to 0.44 m clearance on the return leg.

Change: xacro arg lidar_yaw (default 0.0, so simulation and display keep the
nominal CAD mount) used by lidar_joint; manual_mode.launch.py defaults it to
-0.2225 rad for the real robot and navigation.launch.py forwards it.
manual_mapping/auto_explore inherit it through manual_mode. Roll back with
lidar_yaw:=0.0, no rebuild. Nav2, EKF, AMCL and maps are unchanged.

Contract tests cover the defaults, the forwarding, the URDF default and the
rendered yaw; each of four mutations fails at least one of them.

Co-Authored-By: Claude Opus 5.5 <noreply@anthropic.com>

File: robot/ros2_ws/src/robot_description/urdf/robot.urdf.xacro (robot description, xacro)
@@ -11,4 +11,8 @@
   <xacro:arg name="use_sim" default="true"/>
   <xacro:arg name="use_ros2_control" default="true"/>
+  <!-- Yaw (rad) of lidar_link in base_link. 0 = the CAD/nominal mount, used by
+       simulation and display. The real robot passes its measured calibration
+       from robot_control/launch/manual_mode.launch.py (lidar_yaw). -->
+  <xacro:arg name="lidar_yaw" default="0.0"/>
   <!-- ===== Include cac phan ===== -->
   <xacro:include filename="$(find robot_description)/urdf/common_properties.xacro"/>

File: robot/ros2_ws/src/robot_description/urdf/sensors.xacro (robot description, xacro)
@@ -31,5 +31,5 @@
     <parent link="base_link"/>
     <child  link="lidar_link"/>
-    <origin xyz="${lidar_x} ${lidar_y} ${lidar_z}" rpy="0 0 0"/>
+    <origin xyz="${lidar_x} ${lidar_y} ${lidar_z}" rpy="0 0 $(arg lidar_yaw)"/>
   </joint>
   <gazebo reference="lidar_link">
